File: PCB/SplitHallBoard.kicad_pcb (KiCad board)
At the start: 2 copper layers, 151.2 x 103 mm, 161 parts, among them J1 Display conector, J2 Conn_01x01_Socket, J3 Conn_01x02_Socket, P1 Xiao nRF52840, SW3 EC11N1520401, U0 HX6659ISO-B, U1 HX6659ISO-B, U10 HX6659ISO-B, U11 HX6659ISO-B, U12 HX6659ISO-B, U13 HX6659ISO-B, U14 HX6659ISO-B, U15 HX6659ISO-B, U16 HX6659ISO-B, U17 HX6659ISO-B, U18 HX6659ISO-B, U19 HX6659ISO-B, U2 HX6659ISO-B, U20 HX6659ISO-B, U21 HX6659ISO-B, U22 HX6659ISO-B, U23 HX6659ISO-B, U24 HX6659ISO-B, U25 HX6659ISO-B, U26 HX6659ISO-B, U27 HX6659ISO-B, U28 HX6659ISO-B, U29 HX6659ISO-B, U3 HX6659ISO-B, U30 HX6659ISO-B, U31 HX6659ISO-B, U32 HX6659ISO-B, U33 HX6659ISO-B, U34 HX6659ISO-B, U35 HX6659ISO-B, U36 HX6659ISO-B, U37 HX6659ISO-B, U38 HX6659ISO-B, U39 HX6659ISO-B, U4 HX6659ISO-B, U40 HX6659ISO-B, U41 HX6659ISO-B, U42 HX6659ISO-B, U43 HX6659ISO-B, U44 HX6659ISO-B, U45 HX6659ISO-B, U5 HX6659ISO-B, U6 HX6659ISO-B, U7 HX6659ISO-B, U8 HX6659ISO-B, U9 HX6659ISO-B

Commit message: cleanup
Routing:
- net GND: track 145.6 -> 138.6 mm, vias 63 -> 61
- net K9: track 48.1 -> 51.4 mm
- net MUX2: track 110.4 -> 112.8 mm
- net S2: track 114.2 -> 112.1 mm
- net K15: track 54.6 -> 56.2 mm
- net K12: track 58.9 -> 60.3 mm
- net K8: track 71.7 -> 72.9 mm
- net K6: track 64.8 -> 65.4 mm
- net VBUS: track 179.8 -> 180.4 mm
- net S1: track 124.9 -> 124.7 mm, vias 3 -> 2

Commit message: changes near mux
Routing:
- net GND: track 138.6 -> 142.3 mm, vias 61 -> 62
- net K5: track 83.9 -> 83.1 mm
- net K6: track 65.4 -> 64.8 mm

Commit message: final changes
Parts:
- added H10: MountingHole, MountingHole:MountingHole_2.2mm_M2, F.Cu at (158.0, 62.9)
- added H9: MountingHole, MountingHole:MountingHole_2.2mm_M2, F.Cu at (153.0, 62.9)
Routing:
- net GND: track 142.3 -> 137.1 mm, vias 62 -> 61
- net K12: track 60.3 -> 62.0 mm, vias 0 -> 2
