File: PCB/SplitHallBoard.kicad_sch (KiCad schematic)
At the start: 23 parts, among them J1 Display conector, J2 Conn_01x01_Socket, J3 Conn_01x02_Socket, P1 Xiao nRF52840, SW3 EC11N1520401

Commit message: final changes
Parts:
- added H10, H9: MountingHole, MountingHole:MountingHole_2.2mm_M2, symbol Mechanical:MountingHole
Changed lines of the file:
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@@
+	)
+	(symbol
+		(lib_id "Mechanical:MountingHole")
+		(at 490.22 165.1 0)
+		(unit 1)
+		(exclude_from_sim no)
+		(in_bom yes)
+		(on_board yes)
+		(dnp no)
+		(fields_autoplaced yes)
+		(property "Reference" "H10"
+			(at 492.76 165.0999 0)
+			(effects
+				(font
+					(size 1.27 1.27)
+				)
+				(justify left)
+			)
+		)
+		(property "Value" "MountingHole"
+			(at 492.76 166.37 0)
+			(effects
+				(font
+					(size 1.27 1.27)
+				)
+				(justify left)
+				(hide yes)
+			)
+		)
+		(property "Footprint" "MountingHole:MountingHole_2.2mm_M2"
+			(at 490.22 165.1 0)
+			(effects
+				(font
+					(size 1.27 1.27)
+				)
+				(hide yes)
+			)
+		)
+		(property "Datasheet" "~"
+			(at 490.22 165.1 0)
+			(effects
+				(font
+					(size 1.27 1.27)
+				)
+				(hide yes)
+			)
+		)
+		(property "Description" ""
+			(at 490.22 165.1 0)
+			(effects
+				(font
+					(size 1.27 1.27)
+				)
+				(hide yes)
+			)
+		)
+		(instances
+			(project "SplitHallBoard"
+				(path "/f39183b1-1109-46d9-9ae3-377f71bbe3c7"
+					(reference "H10")
+					(unit 1)
+				)
+			)
+		)
 	)
 	(symbol
@@
 	)
 	(symbol
+		(lib_id "Mechanical:MountingHole")
+		(at 472.44 165.1 0)
+		(unit 1)
+		(exclude_from_sim no)
+		(in_bom yes)
+		(on_board yes)
+		(dnp no)
+		(fields_autoplaced yes)
+		(property "Reference" "H9"
+			(at 474.98 165.0999 0)
+			(effects
+				(font
+					(size 1.27 1.27)
+				)
+				(justify left)
+			)
+		)
+		(property "Value" "MountingHole"
+			(at 474.98 166.37 0)
+			(effects
+				(font
+					(size 1.27 1.27)
+				)
+				(justify left)
+				(hide yes)
+			)
+		)
+		(property "Footprint" "MountingHole:MountingHole_2.2mm_M2"
+			(at 472.44 165.1 0)
+			(effects
+				(font
+					(size 1.27 1.27)
+				)
+				(hide yes)
+			)
+		)
+		(property "Datasheet" "~"
+			(at 472.44 165.1 0)
+			(effects
+				(font
+					(size 1.27 1.27)
+				)
+				(hide yes)
+			)
+		)
+		(property "Description" ""
+			(at 472.44 165.1 0)
+			(effects
+				(font
+					(size 1.27 1.27)
+				)
+				(hide yes)
+			)
+		)
+		(instances
+			(project "SplitHallBoard"
+				(path "/f39183b1-1109-46d9-9ae3-377f71bbe3c7"
+					(reference "H9")
+					(unit 1)
+				)
+			)
+		)
+	)
+	(symbol
 		(lib_id "symbolLib:TCEPQR_0_1")
 		(at 568.96 105.41 0)
@@
 		)
 		(instances
-			(project "+try2"
+			(project "SplitHallBoard"
 				(path "/f39183b1-1109-46d9-9ae3-377f71bbe3c7"
 					(page "7")
@@
 		)
 		(instances
-			(project "+try2"
+			(project "SplitHallBoard"
 				(path "/f39183b1-1109-46d9-9ae3-377f71bbe3c7"
 					(page "20")
@@
 		)
 		(instances
-			(project "+try2"
+			(project "SplitHallBoard"
 				(path "/f39183b1-1109-46d9-9ae3-377f71bbe3c7"
 					(page "19")
@@
 		)
 		(instances
-			(project "+try2"
+			(project "SplitHallBoard"
 				(path "/f39183b1-1109-46d9-9ae3-377f71bbe3c7"
 					(page "12")
@@
 		)
 		(instances
-			(project "+try2"
+			(project "SplitHallBoard"
 				(path "/f39183b1-1109-46d9-9ae3-377f71bbe3c7"
 					(page "16")
@@
 		)
 		(instances
-			(project "+try2"
+			(project "SplitHallBoard"
 				(path "/f39183b1-1109-46d9-9ae3-377f71bbe3c7"
 					(page "24")
@@
 		)
 		(instances
-			(project "+try2"
+			(project "SplitHallBoard"
 				(path "/f39183b1-1109-46d9-9ae3-377f71bbe3c7"
 					(page "6")
@@
 		)
 		(instances
-			(project "+try2"
+			(project "SplitHallBoard"
 				(path "/f39183b1-1109-46d9-9ae3-377f71bbe3c7"
 					(page "21")
@@
 		)
 		(instances
-			(project "+try2"
+			(project "SplitHallBoard"
 				(path "/f39183b1-1109-46d9-9ae3-377f71bbe3c7"
 					(page "18")
@@
 		)
 		(instances
-			(project "+try2"
+			(project "SplitHallBoard"
 				(path "/f39183b1-1109-46d9-9ae3-377f71bbe3c7"
 					(page "15")
@@
 		)
 		(instances
-			(project "+try2"
+			(project "SplitHallBoard"
 				(path "/f39183b1-1109-46d9-9ae3-377f71bbe3c7"
 					(page "22")
@@
 		)
 		(instances
-			(project "+try2"
+			(project "SplitHallBoard"
 				(path "/f39183b1-1109-46d9-9ae3-377f71bbe3c7"
 					(page "23")
@@
 		)
 		(instances
-			(project "+try2"
+			(project "SplitHallBoard"
 				(path "/f39183b1-1109-46d9-9ae3-377f71bbe3c7"
 					(page "2")
@@
 		)
 		(instances
-			(project "+try2"
+			(project "SplitHallBoard"
 				(path "/f39183b1-1109-46d9-9ae3-377f71bbe3c7"
 					(page "5")
@@
 		)
 		(instances
-			(project "+try2"
+			(project "SplitHallBoard"
 				(path "/f39183b1-1109-46d9-9ae3-377f71bbe3c7"
 					(page "11")
@@
 		)
 		(instances
-			(project "+try2"
+			(project "SplitHallBoard"
 				(path "/f39183b1-1109-46d9-9ae3-377f71bbe3c7"
 					(page "8")
@@
 		)
 		(instances
-			(project "+try2"
+			(project "SplitHallBoard"
 				(path "/f39183b1-1109-46d9-9ae3-377f71bbe3c7"
 					(page "10")
@@
 		)
 		(instances
-			(project "+try2"
+			(project "SplitHallBoard"
 				(path "/f39183b1-1109-46d9-9ae3-377f71bbe3c7"
 					(page "13")
@@
 		)
 		(instances
-			(project "+try2"
+			(project "SplitHallBoard"
 				(path "/f39183b1-1109-46d9-9ae3-377f71bbe3c7"
 					(page "9")
@@
 		)
 		(instances
-			(project "+try2"
+			(project "SplitHallBoard"
 				(path "/f39183b1-1109-46d9-9ae3-377f71bbe3c7"
 					(page "17")
@@
 		)
 		(instances
-			(project "+try2"
+			(project "SplitHallBoard"
 				(path "/f39183b1-1109-46d9-9ae3-377f71bbe3c7"
 					(page "14")
@@
 		)
 		(instances
-			(project "+try2"
+			(project "SplitHallBoard"
 				(path "/f39183b1-1109-46d9-9ae3-377f71bbe3c7"
 					(page "3")
@@
 		)
 		(instances
-			(project "+try2"
+			(project "SplitHallBoard"
 				(path "/f39183b1-1109-46d9-9ae3-377f71bbe3c7"
 					(page "4")
